Commit message: Add inverted get-up training and refreshed WF collision asset

File: exts/bipedal_locomotion/bipedal_locomotion/assets/urdf/WF_TRON1A.urdf (robot description, URDF)
Before this commit: robot tron1_wheel_leg, 9 links, 8 joints
Joints:
- joint hip_L_Joint: limit lower=-1.012291 upper=1.396263 effort=20.0 velocity=12.0 -> lower=-1.012291 upper=0.0 effort=20.0 velocity=12.0
- joint hip_R_Joint: limit lower=-1.396263 upper=1.012291 effort=20.0 velocity=12.0 -> lower=0.0 upper=1.012291 effort=20.0 velocity=12.0
